File: SP6N02RTL8211EGigabitEthernetExpansionModule.sch (KiCad schematic (older format))
At the start: 66 parts, among them J1 RJ45(HFJ11-1GO1ERL), P1 HIROSE_120PIN, U1 MCP1825, U2 24AA02E48, U3 RTL8211E-VB, X1 50MHz

Commit message: Converting to pmod connector.
Parts:
- removed P1: HIROSE_120PIN, ~, symbol HIROSE_120PIN
- added PMODD? (x2): PMOD-Device-x2-Type-1A-GPIO, symbol PMOD-Device-x2-Type-1A-GPIO
Connections:
- net labels added: 3V3, SCK, SDA
- wire segments 302 -> 266
- no-connect marks 60 -> 4
Other:
- note added: "Hold SCK down for X ns to start a reset."
- note added: "Need way to share SDA/SCK\nbetween \n * ETH_MDIO/ETH_MDC and \n * MAC_SDA/MAC_SCL"
